Commit message: 删除未使用的模型文件，关闭 FASTLIO Map cloud

File: src/rm_simulation/livox_laser_simulation_RO2/urdf/mid360.xacro (robot description, xacro)
@@ -7,5 +7,5 @@
   <xacro:property name="resolution" value="0.002"/>
   <xacro:property name="noise_mean" value="0.0"/>
-  <xacro:property name="noise_stddev" value="0.01"/>
+  <xacro:property name="noise_stddev" value="0.002"/>
   <xacro:property name="mass" value="0.4" />
   <xacro:property name="length" value="0.1" />

Commit message: 与gitee同步

File: src/rm_simulation/livox_laser_simulation_RO2/urdf/mid360.xacro (robot description, xacro)
@@ -4,5 +4,5 @@
   <xacro:property name="laser_min_range" value="0.1"/>
   <xacro:property name="laser_max_range" value="200.0"/>
-  <xacro:property name="samples" value="40000"/>
+  <xacro:property name="samples" value="30000"/>
   <xacro:property name="resolution" value="0.002"/>
   <xacro:property name="noise_mean" value="0.0"/>

File: src/rm_simulation/pb_rm_simulation/urdf/waking_robot.xacro (robot description, xacro)
@@ -1,17 +1,12 @@
 <?xml version="1.0"?>
 <robot name="robot" xmlns:xacro="http://www.ros.org/wiki/xacro">
-    <xacro:property name="package_name" value="pb_rm_simulation" />
-    <xacro:property name="hokuyo_mesh_path" value="$(find ${package_name})/meshes/hokuyo.dae" />
     <xacro:property name="length_wheel" value="0.05" />
     <xacro:property name="radius_wheel" value="0.06" />
-    <xacro:property name="camera_link" value="0.05" />
     <xacro:property name="PI" value="3.1415926"/>
     <xacro:macro name="default_inertial" params="mass">
         <inertial>
             <mass value="${mass}" />
-            <inertia ixx="0.01" ixy="0.0"
-                        ixz="0.0"
-                        iyy="0.01" iyz="0.0"
-                        izz="0.01" />
+            <inertia ixx="0.01" ixy="0.0" ixz="0.0"
+                    iyy="0.01" iyz="0.0" izz="0.01" />
         </inertial>
     </xacro:macro>
@@ -208,36 +203,4 @@
         </inertial>
     </link>
-    <!-- IMU -->
-    <!-- Camera joint -->
-    <joint name="camera_joint" type="fixed">
-        <axis xyz="0 1 0" />
-        <origin xyz="0 0 0.175" rpy="0 0 0"/>
-        <parent link="base_link"/>
-        <child link="camera_link"/>
-    </joint>
-    <!-- Camera -->
-    <link name="camera_link">
-        <collision>
-            <origin xyz="0 0 0" rpy="0 0 0"/>
-            <geometry>
-                <box size="0.05 0.05 0.05"/>
-            </geometry>
-        </collision>
-        <visual>
-            <origin xyz="0 0 0" rpy="0 0 0"/>
-            <geometry>
-                <box size="0.05 0.05 0.05"/>
-            </geometry>
-            <material name="red">
-                <color rgba="1 0 0 1"/>
-            </material>
-        </visual>
-        <inertial>
-            <mass value="1e-2" />
-            <origin xyz="0 0 0" rpy="0 0 0"/>
-            <inertia ixx="1e-6" ixy="0" ixz="0" iyy="1e-6" iyz="0" izz="1e-6" />
-        </inertial>
-    </link>
-    <!-- camera -->
     <!-- gazebo插件设置相关 -->
     <gazebo reference="base_link">
@@ -256,16 +219,9 @@
         <material>Gazebo/Black</material>
     </gazebo>
-    <!-- ros_control plugin -->
-    <!--   <gazebo>
-    <plugin name="gazebo_ros_control" filename="libgazebo_ros_control.so">
-    <robotNamespace>/robot</robotNamespace>
-    <legacyModeNS> true </legacyModeNS>
-    </plugin>
-    </gazebo> -->
     <!-- Drive controller -->
     <gazebo>
         <plugin name="mecanum_controller" filename="libgazebo_ros_planar_move.so">
             <alwaysOn>true</alwaysOn>
-            <updateRate>100.0</updateRate>
+            <updateRate>20.0</updateRate>
             <robotNamespace>/</robotNamespace>
             <commandTopic>cmd_vel</commandTopic>
@@ -278,5 +234,5 @@
             <wheelSeparation>0.26</wheelSeparation>
             <wheelDiameter>0.12</wheelDiameter>
-            <odometryRate>100.0</odometryRate>
+            <odometryRate>20.0</odometryRate>
             <torque>2</torque>
             <robotBaseFrame>base_footprint</robotBaseFrame>
@@ -313,63 +269,13 @@
         </sensor>
     </gazebo>
-    <!-- 摄像头控制 -->
-    <gazebo reference="camera_link">
-        <material>Gazebo/Orange</material>
-        <gravity>true</gravity>
-        <sensor name="camera_sensor" type="camera">
-            <always_on>true</always_on>
-            <update_rate>30</update_rate>
-            <visualize>false</visualize>
-            <camera name="head">
-                <horizontal_fov>1.3962634</horizontal_fov>
-                <image>
-                    <width>640</width>
-                    <height>480</height>
-                    <format>R8G8B8</format>
-                </image>
-                <clip>
-                    <near>0.1</near>
-                    <far>100</far>
-                </clip>
-                <noise>
-                    <type>gaussian</type>
-                    <mean>0.0</mean>
-                    <stddev>0.007</stddev>
-                </noise>
-            </camera>
-            <plugin filename="libgazebo_ros_camera.so" name="camera_plugin">
-                <alwaysOn>true</alwaysOn>
-                <updateRate>0.0</updateRate>
-                <cameraName>head</cameraName>
-                <imageTopicName>image_raw</imageTopicName>
-                <cameraInfoTopicName>camera_info</cameraInfoTopicName>
-                <frameName>camera_link</frameName>
-                <hackBaseline>0.07</hackBaseline>
-                <distortionK1>0.0</distortionK1>
-                <distortionK2>0.0</distortionK2>
-                <distortionK3>0.0</distortionK3>
-                <distortionT1>0.0</distortionT1>
-                <distortionT2>0.0</distortionT2>
-                <Cx>320.5</Cx>
-                <Cy>240.5</Cy>
-                <Fx>545.5</Fx>
-                <Fy>545.5</Fy>
-                <Tx>0.0</Tx>
-                <Ty>0.0</Ty>
-                <fov>1.3962634</fov>
-                <noise>0.007</noise>
-                <bias>0.0</bias>
-            </plugin>
-        </sensor>
-    </gazebo>
-    <!-- mid360 Laser -->
+    <!-- Livox-Mid360  -->
     <xacro:include filename="$(find ros2_livox_simulation)/urdf/mid360.xacro" />
     <xacro:mid360 name="livox" parent="base_link" topic="mid360">
-        <origin xyz="0 0.0 0.225" rpy="0 0 0"/>
+        <origin xyz="0 0.0 0.175" rpy="0 0 0"/>
     </xacro:mid360>
-    <!-- avia Laser -->
+    <!-- Livox-Avia -->
     <!-- <xacro:include filename="$(find ros2_livox_simulation)/urdf/avia.xacro" />
     <xacro:avia name="livox" parent="base_link" topic="avia">
-        <origin xyz="0 0.0 0.225" rpy="0 0 0"/>
+        <origin xyz="0 0.0 0.175" rpy="0 0 0"/>
     </xacro:avia> -->
 </robot>
